Commit message: Cleanup

File: articutool_description/urdf/articutool.urdf.xacro (robot description, xacro)
@@ -4,13 +4,15 @@
   xmlns:xacro="http://ros.org/wiki/xacro"
 >
-  <xacro:include filename="$(find articutool_description)/urdf/articutool_new.xacro"/>
+  <xacro:arg
+    name="end_effector_tool"
+    default="fork"
+  />
+  <xacro:include filename="$(find articutool_description)/urdf/articutool.xacro"/>
   <xacro:include filename="$(find articutool_description)/urdf/articutool.ros2_control.xacro"/>
-  <link name="world"/>
-  <xacro:articutool parent="world">
-    <origin
-      xyz="0 0 0"
-      rpy="0 0 0"
-    />
-  </xacro:articutool>
+  <xacro:property
+    name="end_effector_tool"
+    value="$(arg end_effector_tool)"
+  />
+  <xacro:articutool end_effector_tool="${end_effector_tool}"/>
   <xacro:articutool_ros2_control name="articutool_ros2_control"/>
 </robot>

File: articutool_description/urdf/articutool_standalone.xacro (robot description, xacro)
@@ -14,5 +14,5 @@
   xmlns:physics="http://playerstage.sourceforge.net/gazebo/xmlschema/#physics"
   xmlns:xacro="http://www.ros.org/wiki/xacro"
-  name="ada"
+  name="articutool"
 >
   <xacro:arg
@@ -22,8 +22,4 @@
   <xacro:include filename="$(find articutool_description)/urdf/articutool.xacro"/>
   <xacro:property
-    name="root"
-    value="root"
-  />
-  <xacro:property
     name="end_effector_tool"
     value="$(arg end_effector_tool)"
