Commit message: Add root roll, pitch, yaw joints and publish joint states to them from estimated orientation quaternion

File: articutool_description/urdf/articutool.xacro (robot description, xacro)
@@ -111,4 +111,46 @@
   >
     <link name="root"/>
+    <link name="root_roll"/>
+    <xacro:articutool_joint
+      joint_name="atool_root_to_roll"
+      type="revolute"
+      parent="root"
+      child="root_roll"
+      joint_axis_xyz="1 0 0"
+      joint_origin_xyz="0 0 0"
+      joint_origin_rpy="0 0 0"
+      joint_velocity_limit="1"
+      joint_torque_limit="1.4"
+      joint_lower_limit="${-J_PI/2}"
+      joint_upper_limit="${J_PI/2}"
+    />
+    <link name="root_pitch"/>
+    <xacro:articutool_joint
+      joint_name="atool_roll_to_pitch"
+      type="revolute"
+      parent="root_roll"
+      child="root_pitch"
+      joint_axis_xyz="0 1 0"
+      joint_origin_xyz="0 0 0"
+      joint_origin_rpy="0 0 0"
+      joint_velocity_limit="1"
+      joint_torque_limit="1.4"
+      joint_lower_limit="${-J_PI/2}"
+      joint_upper_limit="${J_PI/2}"
+    />
+    <link name="root_yaw"/>
+    <xacro:articutool_joint
+      joint_name="atool_pitch_to_yaw"
+      type="revolute"
+      parent="root_pitch"
+      child="root_yaw"
+      joint_axis_xyz="0 0 1"
+      joint_origin_xyz="0 0 0"
+      joint_origin_rpy="0 0 0"
+      joint_velocity_limit="1"
+      joint_torque_limit="1.4"
+      joint_lower_limit="${-J_PI/2}"
+      joint_upper_limit="${J_PI/2}"
+    />
     <xacro:articutool_link
       link_name="atool_handle"
@@ -129,5 +171,5 @@
       joint_name="atool_root_to_handle"
       type="fixed"
-      parent="root"
+      parent="root_yaw"
       child="atool_handle"
       joint_axis_xyz="0 0 1"

Commit message: Remove redundant RPY frames previously used for easy visualization

File: articutool_description/urdf/articutool.xacro (robot description, xacro)
@@ -111,46 +111,4 @@
   >
     <link name="root"/>
-    <link name="root_roll"/>
-    <xacro:articutool_joint
-      joint_name="atool_root_to_roll"
-      type="revolute"
-      parent="root"
-      child="root_roll"
-      joint_axis_xyz="1 0 0"
-      joint_origin_xyz="0 0 0"
-      joint_origin_rpy="0 0 0"
-      joint_velocity_limit="1"
-      joint_torque_limit="1.4"
-      joint_lower_limit="${-J_PI/2}"
-      joint_upper_limit="${J_PI/2}"
-    />
-    <link name="root_pitch"/>
-    <xacro:articutool_joint
-      joint_name="atool_roll_to_pitch"
-      type="revolute"
-      parent="root_roll"
-      child="root_pitch"
-      joint_axis_xyz="0 1 0"
-      joint_origin_xyz="0 0 0"
-      joint_origin_rpy="0 0 0"
-      joint_velocity_limit="1"
-      joint_torque_limit="1.4"
-      joint_lower_limit="${-J_PI/2}"
-      joint_upper_limit="${J_PI/2}"
-    />
-    <link name="root_yaw"/>
-    <xacro:articutool_joint
-      joint_name="atool_pitch_to_yaw"
-      type="revolute"
-      parent="root_pitch"
-      child="root_yaw"
-      joint_axis_xyz="0 0 1"
-      joint_origin_xyz="0 0 0"
-      joint_origin_rpy="0 0 0"
-      joint_velocity_limit="1"
-      joint_torque_limit="1.4"
-      joint_lower_limit="${-J_PI/2}"
-      joint_upper_limit="${J_PI/2}"
-    />
     <xacro:articutool_link
       link_name="atool_handle"
@@ -171,5 +129,5 @@
       joint_name="atool_root_to_handle"
       type="fixed"
-      parent="root_yaw"
+      parent="root"
       child="atool_handle"
       joint_axis_xyz="0 0 1"

Commit message: Add base_parent link parameter. By default, base_parent:=root and a link is created so that the TF tree is properly defined. If base_parent is defined, the link should already exist so that the TF tree is properly defined.

File: articutool_description/urdf/articutool.xacro (robot description, xacro)
@@ -108,7 +108,6 @@
   <xacro:macro
     name="articutool"
-    params="end_effector_tool"
+    params="base_parent end_effector_tool"
   >
-    <link name="root"/>
     <xacro:articutool_link
       link_name="atool_handle"
@@ -129,5 +128,5 @@
       joint_name="atool_root_to_handle"
       type="fixed"
-      parent="root"
+      parent="${base_parent}"
       child="atool_handle"
       joint_axis_xyz="0 0 1"

File: articutool_description/urdf/articutool_standalone.xacro (robot description, xacro)
@@ -25,4 +25,5 @@
     value="$(arg end_effector_tool)"
   />
-  <xacro:articutool end_effector_tool="${end_effector_tool}"/>
+  <link name="root" />
+  <xacro:articutool base_parent="root" end_effector_tool="${end_effector_tool}"/>
 </robot>

File: articutool_moveit/config/articutool.urdf.xacro (robot description, xacro)
@@ -4,4 +4,8 @@
   xmlns:xacro="http://ros.org/wiki/xacro"
 >
+  <xacro:arg
+    name="base_parent"
+    default="root"
+  />
   <xacro:arg
     name="initial_positions_file"
@@ -26,5 +30,12 @@
     value="$(arg end_effector_tool)"
   />
-  <xacro:articutool end_effector_tool="${end_effector_tool}"/>
+  <xacro:property
+    name="base_parent"
+    value="$(arg base_parent)"
+  />
+  <xacro:if value="${base_parent == 'root'}">
+    <link name="${base_parent}" />
+  </xacro:if>
+  <xacro:articutool base_parent="${base_parent}" end_effector_tool="${end_effector_tool}"/>
   <xacro:articutool_ros2_control
     name="articutool_ros2_control"

Commit message: Add imu_frame relative to atool_handle, whose axes encompass the actual axes of measurement as indicated on the silkscreen of the OpenLog Artemis

File: articutool_description/urdf/articutool.xacro (robot description, xacro)
@@ -134,4 +134,10 @@
       joint_origin_rpy="0 0 0"
     />
+    <link name="atool_imu_frame"/>
+    <joint name="atool_handle_to_imu_frame" type="fixed">
+      <parent link="atool_handle"/>
+      <child link="atool_imu_frame"/>
+      <origin xyz="0 0 0" rpy="${-J_PI/2} 0 ${J_PI/2}"/>
+    </joint>
     <xacro:articutool_link
       link_name="atool_electronics_holder"

Commit message: Update IMU frame orientation such that it follows the ENU (East, North, Up) convention where the z-axis points up, opposite to gravity, and rotations about the x and y axes now correspond to roll and pitch respectively

File: articutool_description/urdf/articutool.xacro (robot description, xacro)
@@ -132,5 +132,5 @@
       joint_axis_xyz="0 0 1"
       joint_origin_xyz="0 0 0"
-      joint_origin_rpy="0 0 0"
+      joint_origin_rpy="0 ${-J_PI/2} 0"
     />
     <link name="atool_imu_frame"/>
@@ -138,5 +138,5 @@
       <parent link="atool_handle"/>
       <child link="atool_imu_frame"/>
-      <origin xyz="0 0 0" rpy="${-J_PI/2} 0 ${J_PI/2}"/>
+      <origin xyz="0 0 0" rpy="0 ${-J_PI/2} ${-J_PI}"/>
     </joint>
     <xacro:articutool_link

Commit message: Parameterize scale factor in Xacro

File: articutool_description/urdf/articutool.xacro (robot description, xacro)
@@ -37,4 +37,5 @@
     />
   </xacro:property>
+  <xacro:property name="scale" value="0.001" />
   <xacro:macro
     name="articutool_link"
@@ -46,5 +47,5 @@
           <mesh
             filename="package://articutool_description/meshes/${link_mesh}.stl"
-            scale="0.001 0.001 0.001"
+            scale="${scale} ${scale} ${scale}"
           />
         </geometry>
@@ -57,5 +58,5 @@
           <mesh
             filename="package://articutool_description/meshes/${link_mesh}.stl"
-            scale="0.001 0.001 0.001"
+            scale="${scale} ${scale} ${scale}"
           />
         </geometry>

Commit message: Apply scale factor for joint_origin_xyz

File: articutool_description/urdf/articutool.xacro (robot description, xacro)
@@ -111,4 +111,8 @@
     params="base_parent end_effector_tool joint_origin_xyz:='0 0 0' joint_origin_rpy:='0 0 0'"
   >
+    <xacro:property name="xyz_list" value="${joint_origin_xyz.split(' ')}" />
+    <xacro:property name="scaled_xyz_x" value="${scale * float(xyz_list[0])}" />
+    <xacro:property name="scaled_xyz_y" value="${scale * float(xyz_list[1])}" />
+    <xacro:property name="scaled_xyz_z" value="${scale * float(xyz_list[2])}" />
     <xacro:articutool_link
       link_name="atool_handle"
@@ -132,5 +136,5 @@
       child="atool_handle"
       joint_axis_xyz="0 0 1"
-      joint_origin_xyz="${joint_origin_xyz}"
+      joint_origin_xyz="${scaled_xyz_x} ${scaled_xyz_y} ${scaled_xyz_z}"
       joint_origin_rpy="${joint_origin_rpy}"
     />

Commit message: Run pre-commit

File: articutool_description/urdf/articutool.xacro (robot description, xacro)
@@ -37,5 +37,8 @@
     />
   </xacro:property>
-  <xacro:property name="scale" value="0.001" />
+  <xacro:property
+    name="scale"
+    value="0.001"
+  />
   <xacro:macro
     name="articutool_link"
@@ -111,8 +114,20 @@
     params="base_parent end_effector_tool joint_origin_xyz:='0 0 0' joint_origin_rpy:='0 0 0'"
   >
-    <xacro:property name="xyz_list" value="${joint_origin_xyz.split(' ')}" />
-    <xacro:property name="scaled_xyz_x" value="${scale * float(xyz_list[0])}" />
-    <xacro:property name="scaled_xyz_y" value="${scale * float(xyz_list[1])}" />
-    <xacro:property name="scaled_xyz_z" value="${scale * float(xyz_list[2])}" />
+    <xacro:property
+      name="xyz_list"
+      value="${joint_origin_xyz.split(' ')}"
+    />
+    <xacro:property
+      name="scaled_xyz_x"
+      value="${scale * float(xyz_list[0])}"
+    />
+    <xacro:property
+      name="scaled_xyz_y"
+      value="${scale * float(xyz_list[1])}"
+    />
+    <xacro:property
+      name="scaled_xyz_z"
+      value="${scale * float(xyz_list[2])}"
+    />
     <xacro:articutool_link
       link_name="atool_handle"
@@ -140,8 +155,14 @@
     />
     <link name="atool_imu_frame"/>
-    <joint name="atool_handle_to_imu_frame" type="fixed">
+    <joint
+      name="atool_handle_to_imu_frame"
+      type="fixed"
+    >
       <parent link="atool_handle"/>
       <child link="atool_imu_frame"/>
-      <origin xyz="0 0 0" rpy="0 ${-J_PI/2} ${-J_PI}"/>
+      <origin
+        xyz="0 0 0"
+        rpy="0 ${-J_PI/2} ${-J_PI}"
+      />
     </joint>
     <xacro:articutool_link

File: articutool_description/urdf/articutool_standalone.xacro (robot description, xacro)
@@ -25,5 +25,8 @@
     value="$(arg end_effector_tool)"
   />
-  <link name="root" />
-  <xacro:articutool base_parent="root" end_effector_tool="${end_effector_tool}"/>
+  <link name="root"/>
+  <xacro:articutool
+    base_parent="root"
+    end_effector_tool="${end_effector_tool}"
+  />
 </robot>

File: articutool_moveit/config/articutool.urdf.xacro (robot description, xacro)
@@ -47,7 +47,12 @@
   />
   <xacro:if value="${base_parent == 'root'}">
-    <link name="${base_parent}" />
+    <link name="${base_parent}"/>
   </xacro:if>
-  <xacro:articutool base_parent="${base_parent}" end_effector_tool="${end_effector_tool}" joint_origin_xyz="$(arg joint_origin_xyz)" joint_origin_rpy="$(arg joint_origin_rpy)"/>
+  <xacro:articutool
+    base_parent="${base_parent}"
+    end_effector_tool="${end_effector_tool}"
+    joint_origin_xyz="$(arg joint_origin_xyz)"
+    joint_origin_rpy="$(arg joint_origin_rpy)"
+  />
   <xacro:if value="$(arg launch_controllers)">
     <xacro:articutool_ros2_control

Commit message: Add dummy configuration for Articutool xacro. This should only be used if the system that the Xacro is loaded in does not intend to be responsible for actuating the Articutool's joints. For instance, when the parent system (e.g. ADA) wants to maintain a dummy copy of the Articutool for motion planning and collision avoidance.

File: articutool_description/urdf/articutool.xacro (robot description, xacro)
@@ -77,5 +77,5 @@
   <xacro:macro
     name="articutool_joint"
-    params="joint_name type parent child joint_axis_xyz joint_origin_xyz joint_origin_rpy joint_lower_limit:=${default_value} joint_upper_limit:=${default_value} joint_velocity_limit:=${default_value} joint_torque_limit:=${default_value}"
+    params="joint_name type parent child joint_axis_xyz joint_origin_xyz joint_origin_rpy joint_lower_limit:=${default_value} joint_upper_limit:=${default_value} joint_velocity_limit:=${default_value} joint_torque_limit:=${default_value} create_mimic:=false mimic_parent:=${base_parent}"
   >
     <joint
@@ -108,9 +108,12 @@
         friction="0.0"
       />
+      <xacro:if value="${create_mimic}">
+        <mimic joint="${mimic_parent}"/>
+      </xacro:if>
     </joint>
   </xacro:macro>
   <xacro:macro
     name="articutool"
-    params="base_parent end_effector_tool joint_origin_xyz:='0 0 0' joint_origin_rpy:='0 0 0'"
+    params="base_parent end_effector_tool joint_origin_xyz:='0 0 0' joint_origin_rpy:='0 0 0' dummy:='false'"
   >
     <xacro:property
@@ -215,17 +218,65 @@
       />
     </xacro:articutool_link>
-    <xacro:articutool_joint
-      joint_name="atool_joint1"
-      type="revolute"
-      parent="atool_base"
-      child="atool_link1"
-      joint_axis_xyz="0 0 -1"
-      joint_origin_xyz="0 0 ${scale * 55}"
-      joint_origin_rpy="${-J_PI/2} 0 0"
-      joint_lower_limit="${-J_PI/2}"
-      joint_upper_limit="${J_PI/2}"
-      joint_velocity_limit="1"
-      joint_torque_limit="1.4"
-    />
+    <link name="atool_joint1_terminator_link"/>
+    <xacro:if value="${dummy}">
+      <xacro:articutool_joint
+        joint_name="atool_joint1"
+        type="revolute"
+        parent="atool_base"
+        child="atool_joint1_terminator_link"
+        joint_axis_xyz="0 0 -1"
+        joint_origin_xyz="0 0 ${scale * 55}"
+        joint_origin_rpy="${-J_PI/2} 0 0"
+        joint_lower_limit="${-J_PI/2}"
+        joint_upper_limit="${J_PI/2}"
+        joint_velocity_limit="1"
+        joint_torque_limit="1.4"
+      />
+      <xacro:articutool_joint
+        joint_name="atool_joint1_mimic"
+        type="revolute"
+        parent="atool_base"
+        child="atool_link1"
+        joint_axis_xyz="0 0 -1"
+        joint_origin_xyz="0 0 ${scale * 55}"
+        joint_origin_rpy="${-J_PI/2} 0 0"
+        joint_lower_limit="${-J_PI/2}"
+        joint_upper_limit="${J_PI/2}"
+        joint_velocity_limit="1"
+        joint_torque_limit="1.4"
+        create_mimic="true"
+        mimic_parent="atool_joint1"
+      />
+    </xacro:if>
+    <xacro:unless value="${dummy}">
+      <xacro:articutool_joint
+        joint_name="atool_joint1"
+        type="revolute"
+        parent="atool_base"
+        child="atool_link1"
+        joint_axis_xyz="0 0 -1"
+        joint_origin_xyz="0 0 ${scale * 55}"
+        joint_origin_rpy="${-J_PI/2} 0 0"
+        joint_lower_limit="${-J_PI/2}"
+        joint_upper_limit="${J_PI/2}"
+        joint_velocity_limit="1"
+        joint_torque_limit="1.4"
+      />
+      <xacro:articutool_joint
+        joint_name="atool_joint1_mimic"
+        type="revolute"
+        parent="atool_base"
+        child="atool_joint1_terminator_link"
+        joint_axis_xyz="0 0 -1"
+        joint_origin_xyz="0 0 ${scale * 55}"
+        joint_origin_rpy="${-J_PI/2} 0 0"
+        joint_lower_limit="${-J_PI/2}"
+        joint_upper_limit="${J_PI/2}"
+        joint_velocity_limit="1"
+        joint_torque_limit="1.4"
+        create_mimic="true"
+        mimic_parent="atool_joint1"
+      />
+    </xacro:unless>
     <xacro:articutool_link
       link_name="atool_motor_link"
@@ -277,17 +328,65 @@
       <xacro:insert_block name="default_inertial"/>
     </xacro:articutool_link>
-    <xacro:articutool_joint
-      joint_name="atool_joint2"
-      type="revolute"
-      parent="atool_link2"
-      child="atool_ft_adapter"
-      joint_axis_xyz="0 0 1"
-      joint_origin_xyz="0 0 ${scale * 19}"
-      joint_origin_rpy="0 0 0"
-      joint_lower_limit="${-J_PI}"
-      joint_upper_limit="${J_PI}"
-      joint_velocity_limit="1"
-      joint_torque_limit="1.4"
-    />
+    <link name="atool_joint2_terminator_link"/>
+    <xacro:if value="${dummy}">
+      <xacro:articutool_joint
+        joint_name="atool_joint2"
+        type="revolute"
+        parent="atool_link2"
+        child="atool_joint2_terminator_link"
+        joint_axis_xyz="0 0 1"
+        joint_origin_xyz="0 0 ${scale * 19}"
+        joint_origin_rpy="0 0 0"
+        joint_lower_limit="${-J_PI}"
+        joint_upper_limit="${J_PI}"
+        joint_velocity_limit="1"
+        joint_torque_limit="1.4"
+      />
+      <xacro:articutool_joint
+        joint_name="atool_joint2_mimic"
+        type="revolute"
+        parent="atool_link2"
+        child="atool_ft_adapter"
+        joint_axis_xyz="0 0 1"
+        joint_origin_xyz="0 0 ${scale * 19}"
+        joint_origin_rpy="0 0 0"
+        joint_lower_limit="${-J_PI}"
+        joint_upper_limit="${J_PI}"
+        joint_velocity_limit="1"
+        joint_torque_limit="1.4"
+        create_mimic="true"
+        mimic_parent="atool_joint2"
+      />
+    </xacro:if>
+    <xacro:unless value="${dummy}">
+      <xacro:articutool_joint
+        joint_name="atool_joint2"
+        type="revolute"
+        parent="atool_link2"
+        child="atool_ft_adapter"
+        joint_axis_xyz="0 0 1"
+        joint_origin_xyz="0 0 ${scale * 19}"
+        joint_origin_rpy="0 0 0"
+        joint_lower_limit="${-J_PI}"
+        joint_upper_limit="${J_PI}"
+        joint_velocity_limit="1"
+        joint_torque_limit="1.4"
+      />
+      <xacro:articutool_joint
+        joint_name="atool_joint2_mimic"
+        type="revolute"
+        parent="atool_link2"
+        child="atool_joint2_terminator_link"
+        joint_axis_xyz="0 0 1"
+        joint_origin_xyz="0 0 ${scale * 19}"
+        joint_origin_rpy="0 0 0"
+        joint_lower_limit="${-J_PI}"
+        joint_upper_limit="${J_PI}"
+        joint_velocity_limit="1"
+        joint_torque_limit="1.4"
+        create_mimic="true"
+        mimic_parent="atool_joint2"
+      />
+    </xacro:unless>
     <xacro:articutool_link
       link_name="ft"
