Commit message: Remove dummy and mimic parameters

File: articutool_description/urdf/articutool.xacro (robot description, xacro)
@@ -77,5 +77,5 @@
   <xacro:macro
     name="articutool_joint"
-    params="joint_name type parent child joint_axis_xyz joint_origin_xyz joint_origin_rpy joint_lower_limit:=${default_value} joint_upper_limit:=${default_value} joint_velocity_limit:=${default_value} joint_torque_limit:=${default_value} create_mimic:=false mimic_parent:=${base_parent}"
+    params="joint_name type parent child joint_axis_xyz joint_origin_xyz joint_origin_rpy joint_lower_limit:=${default_value} joint_upper_limit:=${default_value} joint_velocity_limit:=${default_value} joint_torque_limit:=${default_value}"
   >
     <joint
@@ -108,12 +108,9 @@
         friction="0.0"
       />
-      <xacro:if value="${create_mimic}">
-        <mimic joint="${mimic_parent}"/>
-      </xacro:if>
     </joint>
   </xacro:macro>
   <xacro:macro
     name="articutool"
-    params="base_parent end_effector_tool joint_origin_xyz:='0 0 0' joint_origin_rpy:='0 0 0' dummy:='false'"
+    params="base_parent end_effector_tool joint_origin_xyz:='0 0 0' joint_origin_rpy:='0 0 0'"
   >
     <xacro:property
@@ -218,65 +215,17 @@
       />
     </xacro:articutool_link>
-    <link name="atool_joint1_terminator_link"/>
-    <xacro:if value="${dummy}">
-      <xacro:articutool_joint
-        joint_name="atool_joint1"
-        type="revolute"
-        parent="atool_base"
-        child="atool_joint1_terminator_link"
-        joint_axis_xyz="0 0 -1"
-        joint_origin_xyz="0 0 ${scale * 55}"
-        joint_origin_rpy="${-J_PI/2} 0 0"
-        joint_lower_limit="${-J_PI/2}"
-        joint_upper_limit="${J_PI/2}"
-        joint_velocity_limit="1"
-        joint_torque_limit="1.4"
-      />
-      <xacro:articutool_joint
-        joint_name="atool_joint1_mimic"
-        type="revolute"
-        parent="atool_base"
-        child="atool_link1"
-        joint_axis_xyz="0 0 -1"
-        joint_origin_xyz="0 0 ${scale * 55}"
-        joint_origin_rpy="${-J_PI/2} 0 0"
-        joint_lower_limit="${-J_PI/2}"
-        joint_upper_limit="${J_PI/2}"
-        joint_velocity_limit="1"
-        joint_torque_limit="1.4"
-        create_mimic="true"
-        mimic_parent="atool_joint1"
-      />
-    </xacro:if>
-    <xacro:unless value="${dummy}">
-      <xacro:articutool_joint
-        joint_name="atool_joint1"
-        type="revolute"
-        parent="atool_base"
-        child="atool_link1"
-        joint_axis_xyz="0 0 -1"
-        joint_origin_xyz="0 0 ${scale * 55}"
-        joint_origin_rpy="${-J_PI/2} 0 0"
-        joint_lower_limit="${-J_PI/2}"
-        joint_upper_limit="${J_PI/2}"
-        joint_velocity_limit="1"
-        joint_torque_limit="1.4"
-      />
-      <xacro:articutool_joint
-        joint_name="atool_joint1_mimic"
-        type="revolute"
-        parent="atool_base"
-        child="atool_joint1_terminator_link"
-        joint_axis_xyz="0 0 -1"
-        joint_origin_xyz="0 0 ${scale * 55}"
-        joint_origin_rpy="${-J_PI/2} 0 0"
-        joint_lower_limit="${-J_PI/2}"
-        joint_upper_limit="${J_PI/2}"
-        joint_velocity_limit="1"
-        joint_torque_limit="1.4"
-        create_mimic="true"
-        mimic_parent="atool_joint1"
-      />
-    </xacro:unless>
+    <xacro:articutool_joint
+      joint_name="atool_joint1"
+      type="revolute"
+      parent="atool_base"
+      child="atool_link1"
+      joint_axis_xyz="0 0 -1"
+      joint_origin_xyz="0 0 ${scale * 55}"
+      joint_origin_rpy="${-J_PI/2} 0 0"
+      joint_lower_limit="${-J_PI/2}"
+      joint_upper_limit="${J_PI/2}"
+      joint_velocity_limit="1"
+      joint_torque_limit="1.4"
+    />
     <xacro:articutool_link
       link_name="atool_motor_link"
@@ -328,65 +277,17 @@
       <xacro:insert_block name="default_inertial"/>
     </xacro:articutool_link>
-    <link name="atool_joint2_terminator_link"/>
-    <xacro:if value="${dummy}">
-      <xacro:articutool_joint
-        joint_name="atool_joint2"
-        type="revolute"
-        parent="atool_link2"
-        child="atool_joint2_terminator_link"
-        joint_axis_xyz="0 0 1"
-        joint_origin_xyz="0 0 ${scale * 19}"
-        joint_origin_rpy="0 0 0"
-        joint_lower_limit="${-J_PI}"
-        joint_upper_limit="${J_PI}"
-        joint_velocity_limit="1"
-        joint_torque_limit="1.4"
-      />
-      <xacro:articutool_joint
-        joint_name="atool_joint2_mimic"
-        type="revolute"
-        parent="atool_link2"
-        child="atool_ft_adapter"
-        joint_axis_xyz="0 0 1"
-        joint_origin_xyz="0 0 ${scale * 19}"
-        joint_origin_rpy="0 0 0"
-        joint_lower_limit="${-J_PI}"
-        joint_upper_limit="${J_PI}"
-        joint_velocity_limit="1"
-        joint_torque_limit="1.4"
-        create_mimic="true"
-        mimic_parent="atool_joint2"
-      />
-    </xacro:if>
-    <xacro:unless value="${dummy}">
-      <xacro:articutool_joint
-        joint_name="atool_joint2"
-        type="revolute"
-        parent="atool_link2"
-        child="atool_ft_adapter"
-        joint_axis_xyz="0 1 0"
-        joint_origin_xyz="0 0 ${scale * 23}"
-        joint_origin_rpy="${J_PI/2} 0 0"
-        joint_lower_limit="${-J_PI}"
-        joint_upper_limit="${J_PI}"
-        joint_velocity_limit="1"
-        joint_torque_limit="1.4"
-      />
-      <xacro:articutool_joint
-        joint_name="atool_joint2_mimic"
-        type="revolute"
-        parent="atool_link2"
-        child="atool_joint2_terminator_link"
-        joint_axis_xyz="0 0 1"
-        joint_origin_xyz="0 0 ${scale * 19}"
-        joint_origin_rpy="0 0 0"
-        joint_lower_limit="${-J_PI}"
-        joint_upper_limit="${J_PI}"
-        joint_velocity_limit="1"
-        joint_torque_limit="1.4"
-        create_mimic="true"
-        mimic_parent="atool_joint2"
-      />
-    </xacro:unless>
+    <xacro:articutool_joint
+      joint_name="atool_joint2"
+      type="revolute"
+      parent="atool_link2"
+      child="atool_ft_adapter"
+      joint_axis_xyz="0 1 0"
+      joint_origin_xyz="0 0 ${scale * 23}"
+      joint_origin_rpy="${J_PI/2} 0 0"
+      joint_lower_limit="${-J_PI}"
+      joint_upper_limit="${J_PI}"
+      joint_velocity_limit="1"
+      joint_torque_limit="1.4"
+    />
     <xacro:articutool_link
       link_name="ft"

Commit message: Add configuration file to define xyz origins for tool_tip frame. This is useful when defining new tool tips since the exact origin will differ by the particular model

File: articutool_description/urdf/articutool.xacro (robot description, xacro)
@@ -41,4 +41,17 @@
     value="0.001"
   />
+  <xacro:arg
+    name="tool_tip_configs_file_arg"
+    default="$(find articutool_description)/config/tool_tip_configurations.yaml"
+  />
+  <xacro:property name="tool_tip_configs_file" value="$(arg tool_tip_configs_file_arg)"/>
+  <xacro:property name="tool_tip_configs" value="${xacro.load_yaml(tool_tip_configs_file)}"/>
+  <xacro:property
+    name="current_tool_specific_config"
+    value="${tool_tip_configs[end_effector_tool] if end_effector_tool in tool_tip_configs else tool_tip_configs['default_tool']}"
+    />
+  <xacro:property name="tool_tip_x_val" value="${scale * current_tool_specific_config['x_mm']}"/>
+  <xacro:property name="tool_tip_y_val" value="${scale * current_tool_specific_config['y_mm']}"/>
+  <xacro:property name="tool_tip_z_val" value="${scale * current_tool_specific_config['z_mm']}"/>
   <xacro:macro
     name="articutool_link"
@@ -347,5 +360,5 @@
       <origin
         rpy="0 0 ${-J_PI/2}"
-        xyz="${scale * 7} 0 ${scale * 70}"
+        xyz="${tool_tip_x_val} ${tool_tip_y_val} ${tool_tip_z_val}"
       />
     </joint>
