Commit message: Run pre-commit

File: articutool_moveit/config/articutool.ros2_control.xacro (robot description, xacro)
@@ -5,5 +5,8 @@
     params="name initial_positions_file sim u2d2_port"
   >
-    <xacro:property name="initial_positions" value="${xacro.load_yaml(initial_positions_file)['initial_positions']}"/>
+    <xacro:property
+      name="initial_positions"
+      value="${xacro.load_yaml(initial_positions_file)['initial_positions']}"
+    />
     <ros2_control
       name="${name}"
@@ -30,8 +33,8 @@
         </state_interface>
         <state_interface name="velocity">
-            <param name="initial_value">0.0</param>
+          <param name="initial_value">0.0</param>
         </state_interface>
         <state_interface name="effort">
-            <param name="initial_value">0.0</param>
+          <param name="initial_value">0.0</param>
         </state_interface>
       </joint>
@@ -44,8 +47,8 @@
         </state_interface>
         <state_interface name="velocity">
-            <param name="initial_value">0.0</param>
+          <param name="initial_value">0.0</param>
         </state_interface>
         <state_interface name="effort">
-            <param name="initial_value">0.0</param>
+          <param name="initial_value">0.0</param>
         </state_interface>
       </joint>

File: articutool_moveit/config/articutool.urdf.xacro (robot description, xacro)
@@ -4,11 +4,20 @@
   xmlns:xacro="http://ros.org/wiki/xacro"
 >
-  <xacro:arg name="initial_positions_file" default="initial_positions.yaml" />
-  <xacro:arg name="sim" default="real" />
+  <xacro:arg
+    name="initial_positions_file"
+    default="initial_positions.yaml"
+  />
+  <xacro:arg
+    name="sim"
+    default="real"
+  />
   <xacro:arg
     name="end_effector_tool"
     default="fork"
   />
-  <xacro:arg name="u2d2_port" default="/dev/u2d2" />
+  <xacro:arg
+    name="u2d2_port"
+    default="/dev/u2d2"
+  />
   <xacro:include filename="$(find articutool_description)/urdf/articutool.xacro"/>
   <xacro:include filename="articutool.ros2_control.xacro"/>
@@ -18,4 +27,9 @@
   />
   <xacro:articutool end_effector_tool="${end_effector_tool}"/>
-  <xacro:articutool_ros2_control name="articutool_ros2_control" initial_positions_file="$(arg initial_positions_file)" sim="$(arg sim)" u2d2_port="$(arg u2d2_port)"/>
+  <xacro:articutool_ros2_control
+    name="articutool_ros2_control"
+    initial_positions_file="$(arg initial_positions_file)"
+    sim="$(arg sim)"
+    u2d2_port="$(arg u2d2_port)"
+  />
 </robot>
